Commit message: added a manual broadcaster for the headlink and the roll_M1_link

File: my_mira_description/urdf/mira.urdf (robot description, URDF)
Before this commit: robot mira, 2 links, 1 joints
Links:
- added link camera_link; visual box size=0.0005 0.0005 0.0005
- added link head_link; visual sphere radius=0.06
- added link left_eye_link; visual cylinder length=0.00525 radius=0.00525
- added link pitch_M2_link; visual cylinder length=0.001 radius=0.005
- added link right_eye_link; visual cylinder length=0.00525 radius=0.00525
- added link yaw_M3_link; visual cylinder length=0.001 radius=0.005
- link roll_M1_link: geometry visual cylinder length=0.001 radius=0.005
Joints:
- removed joint roll_join
- added joint base_head_joint: type fixed, parent yaw_M3_link, child head_link
- added joint camera_head_joint: type fixed, parent head_link, child camera_link
- added joint left_head_joint: type fixed, parent head_link, child left_eye_link
- added joint pitch_joint: type revolute, parent base_link, child pitch_M2_link, origin xyz=0.0023 0 -0.0005 rpy=0 0 0, axis 0 1 0, limit lower=-0.2 upper=0.2 effort=0.1 velocity=0.005
- added joint right_head_joint: type fixed, parent head_link, child right_eye_link
- added joint roll_joint: type revolute, parent base_link, child roll_M1_link, origin xyz=0.0023 0 -0.0005 rpy=0 0 0, axis 1 0 0, limit lower=-0.2 upper=0.2 effort=0.1 velocity=0.005
- added joint yaw_joint: type revolute, parent base_link, child yaw_M3_link, origin xyz=0.0023 0 -0.0005 rpy=0 0 0, axis 0 0 1, limit lower=-0.2 upper=0.2 effort=0.1 velocity=0.005

Commit message: added the capavility for mira to pitch and yaw

File: my_mira_description/urdf/mira.urdf (robot description, URDF)
Before this commit: robot mira, 8 links, 7 joints
Joints:
- removed joint base_head_joint
- removed joint pitch_joint
- removed joint yaw_joint
- added joint pitch_head_joint: type fixed, parent pitch_M2_link, child head_link
- added joint roll_head_joint: type fixed, parent roll_M1_link, child head_link
- added joint roll_pitch_joint: type revolute, parent roll_M1_link, child pitch_M2_link, origin xyz=0 0 0 rpy=0 0 0, axis 0 1 0, limit lower=-0.44 upper=0.44 effort=0.1 velocity=0.005
- added joint yaw_head_joint: type fixed, parent yaw_M3_link, child head_link
- added joint yaw_pitch_joint: type revolute, parent pitch_M2_link, child yaw_M3_link, origin xyz=0 0 0 rpy=0 0 0, axis 0 0 1, limit lower=-0.44 upper=0.44 effort=0.1 velocity=0.005
- joint roll_joint: limit lower=-0.2 upper=0.2 effort=0.1 velocity=0.005 -> lower=-0.22 upper=0.22 effort=0.1 velocity=0.005
