Commit message: added a file to calculate simple inertial moments and finished the gurdy model without the controllers

File: my_gurdy_description/urdf/gurdy.urdf (robot description, URDF)
Before this commit: robot gurdy, 11 links, 10 joints
Links:
- link base_link: mass None -> 0.0; geometry collision box size=0.01 0.01 0.01; visual box size=0.01 0.01 0.01
- link footM1_link: mass None -> 0.01; geometry collision sphere radius=0.006; visual sphere radius=0.006
- link footM2_link: mass None -> 0.01; geometry collision sphere radius=0.006; visual sphere radius=0.006
- link footM3_link: mass None -> 0.01; geometry collision sphere radius=0.006; visual sphere radius=0.006
- link head_link: mass None -> 0.01
- link lowerleg_M1_link: mass None -> 0.01; geometry collision cylinder length=0.06 radius=0.0025; visual mesh filename=package://my_gurdy_description/models/meshes/gurdy_lowerleg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
- link lowerleg_M2_link: mass None -> 0.01; geometry collision cylinder length=0.06 radius=0.0025; visual mesh filename=package://my_gurdy_description/models/meshes/gurdy_lowerleg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
- link lowerleg_M3_link: mass None -> 0.01; geometry collision cylinder length=0.06 radius=0.0025; visual mesh filename=package://my_gurdy_description/models/meshes/gurdy_lowerleg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
- link upperleg_M1_link: mass None -> 0.01; geometry collision cylinder length=0.06 radius=0.0025; visual mesh filename=package://my_gurdy_description/models/meshes/gurdy_higherle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
- link upperleg_M2_link: mass None -> 0.01; geometry collision cylinder length=0.06 radius=0.0025; visual mesh filename=package://my_gurdy_description/models/meshes/gurdy_higherle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
- link upperleg_M3_link: mass None -> 0.01; geometry collision cylinder length=0.06 radius=0.0025; visual mesh filename=package://my_gurdy_description/models/meshes/gurdy_higherle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

Commit message: finished gurdy and downloaded a code that runs it to verify my model was right

File: my_gurdy_description/urdf/gurdy.urdf (robot description, URDF)
Before this commit: robot gurdy, 11 links, 10 joints
Joints:
- joint head_upperlegM1_joint: limit lower=-1.5707 upper=0.0 effort=0.0 velocity=0.005 -> lower=-1.5707 upper=0.0 effort=1.0 velocity=0.005
- joint head_upperlegM2_joint: limit lower=-1.5707 upper=0.0 effort=0.0 velocity=0.005 -> lower=-1.5707 upper=0.0 effort=1.0 velocity=0.005
- joint head_upperlegM3_joint: limit lower=-1.5707 upper=0.0 effort=0.0 velocity=0.005 -> lower=-1.5707 upper=0.0 effort=1.0 velocity=0.005
- joint upperlegM1_lowerlegM1_joint: limit lower=-3 upper=1.5707 effort=0.0 velocity=0.005 -> lower=-3 upper=1.5707 effort=1.0 velocity=0.005
- joint upperlegM2_lowerlegM2_joint: limit lower=-3 upper=1.5707 effort=0.0 velocity=0.005 -> lower=-3 upper=1.5707 effort=1.0 velocity=0.005
- joint upperlegM3_lowerlegM3_joint: limit lower=-3 upper=1.5707 effort=0.0 velocity=0.005 -> lower=-3 upper=1.5707 effort=1.0 velocity=0.005
